Commit message: added lightsaber

File: urdf/iiwa7.urdf (robot description, URDF)
Before this commit: robot iiwa7, 10 links, 9 joints
Links:
- added link lightsaber; collision mesh filename=package://me133a-final-project/meshes/iiwa7/collision/light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 scale=0.001 0.001 0.001; visual mesh filename=package://me133a-final-project/meshes/iiwa7/visual/lightsab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 scale=0.001 0.001 0.001
- added link lightsaber_blade; collision cylinder length=0.8 radius=0.015; visual cylinder length=0.8 radius=0.015
Joints:
- added joint lightsaber_blade_joint: type fixed, parent lightsaber, child lightsaber_blade, origin xyz=0 0 0.15 rpy=0 0 0
- added joint lightsaber_joint: type fixed, parent iiwa_link_ee, child lightsaber, origin xyz=0 0 0.045 rpy=0 0 0

Commit message: kinda working with two points

File: urdf/iiwa7.urdf (robot description, URDF)
Before this commit: robot iiwa7, 12 links, 11 joints
Links:
- removed link lightsaber
- added link lightsaber_base; collision mesh filename=package://me133a-final-project/meshes/iiwa7/collision/light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 scale=0.001 0.001 0.001; visual mesh filename=package://me133a-final-project/meshes/iiwa7/visual/lightsab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 scale=0.001 0.001 0.001
Joints:
- joint lightsaber_blade_joint: origin xyz=0 0 0.15 rpy=0 0 0 -> xyz=0 0 0.2 rpy=0 0 0; parent lightsaber -> lightsaber_base
- joint lightsaber_joint: child lightsaber -> lightsaber_base; origin xyz=0 0 0.045 rpy=0 0 0 -> xyz=0 0 0.02 rpy=0 1.5707963267948966 0

Commit message: converted to other methbod

File: urdf/iiwa7.urdf (robot description, URDF)
Before this commit: robot iiwa7, 12 links, 11 joints
Links:
- added link lightsaber_blade_base; collision cylinder length=0.8 radius=0.015; visual cylinder length=0.8 radius=0.015
- added link lightsaber_blade_end
- added link lightsaber_blade_pan
- added link lightsaber_blade_tilt
- link lightsaber_blade: geometry 
Joints:
- added joint light_saber_blade_end: type prismatic, parent lightsaber_blade_tilt, child lightsaber_blade_end, origin xyz=0 0 0 rpy=0 0 0, axis 0 0 1, limit lower=0.0 upper=10.0 effort=1000.0 velocity=0.5
- added joint light_saber_blade_len: type prismatic, parent lightsaber_blade_base, child lightsaber_blade, origin xyz=0 0 0 rpy=0 0 0, axis 0 0 1, limit lower=0.0 upper=0.8 effort=1000.0 velocity=0.5
- added joint light_saber_blade_pan: type continuous, parent lightsaber_blade, child lightsaber_blade_pan, origin xyz=0 0 0 rpy=0 0 0, axis 0 0 1
- added joint light_saber_blade_tilt: type continuous, parent lightsaber_blade_pan, child lightsaber_blade_tilt, origin xyz=0 0 0 rpy=0 0 0, axis 0 1 0
- joint lightsaber_blade_joint: child lightsaber_blade -> lightsaber_blade_base
